File: ET-Abschlussgadget_2023/ET-Abschlussgadget_2023.kicad_sch (KiCad schematic)
At the start: 24 parts, among them J1 PB0, J2 PB1, J3 UPDI / RESET, J4 EXTCLK, J5 EXTCLK, J6 EXTCLK, SW1 ON/OFF, U1 ATtiny414-SS

Commit message: Changed button-footprint, moved resistors & capacitors from 0805 to 0603, minor tweaks
Parts:
- C1: footprint Capacitor_SMD:C_0805_2012Metric_Pad1.18x1.45mm_HandSolder -> Capacitor_SMD:C_0603_1608Metric_Pad1.08x0.95mm_HandSolder
- R1, R2, R3, R4, R5, R6, R7: footprint Resistor_SMD:R_0805_2012Metric_Pad1.20x1.40mm_HandSolder -> Resistor_SMD:R_0603_1608Metric_Pad0.98x0.95mm_HandSolder
- SW1: footprint Button_Switch_SMD:SW_SPDT_PCM12 -> Button_Switch_SMD:DEALON_MK-12D04-G2
Connections:
- net Cap_Pad: no longer U1.12 (PA2)
- net Cap_Pad / ADC1: now also U1.12 (PA2)
- net GND: now also D1.1 (K), D2.1 (K), D3.1 (K), D4.1 (K), D5.1 (K), D6.1 (K); no longer D1.2 (A), D2.2 (A), D3.2 (A), D4.2 (A), D5.2 (A), D6.2 (A)
- net VCC: now also SW1.3 (C); no longer SW1.1 (A)
- net at R3.2: now also D3.2 (A); no longer D3.1 (K)
- net at R6.1: now also D5.2 (A); no longer D5.1 (K)
- net at R2.1: now also D2.2 (A); no longer D2.1 (K)
- net at R7.1: now also D6.2 (A); no longer D6.1 (K)
- net at R4.2: now also D4.2 (A); no longer D4.1 (K)
- net at R1.1: now also D1.2 (A); no longer D1.1 (K)
Other:
- moved on the sheet: C1, D1, D2, D3, D4, D5, D6

Commit message: Updated switch & battery holder footprint, adjusted manual BOM
Parts:
- BT1: footprint Battery:BatteryHolder_Keystone_3002_1x2032 -> easyeda2kicad:BAT-SMD_CR2032-3V
- SW1: footprint Button_Switch_SMD:DEALON_MK-12D04-G2 -> easyeda2kicad:SW-TH_MSK12C02
Connections:
- net VCC: now also SW1.1 (A); no longer SW1.3 (C)
Other:
- moved on the sheet: C1
Changed lines of the file:
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@@
 (kicad_sch (version 20230121) (generator eeschema)
   (paper "A4")
-  (junction (at 78.74 87.63) (diameter 0) (color 0 0 0 0)
+  (junction (at 78.74 82.55) (diameter 0) (color 0 0 0 0)
   )
   (junction (at 166.37 100.33) (diameter 0) (color 0 0 0 0)
@@
   (junction (at 187.96 85.09) (diameter 0) (color 0 0 0 0)
   )
-  (no_connect (at 74.93 82.55))
+  (no_connect (at 74.93 87.63))
   (wire (pts (xy 181.61 82.55) (xy 166.37 82.55))
     (stroke (width 0) (type default))
@@
     (stroke (width 0) (type default))
   )
-  (wire (pts (xy 78.74 87.63) (xy 83.82 87.63))
+  (wire (pts (xy 78.74 82.55) (xy 83.82 82.55))
     (stroke (width 0) (type default))
   )
@@
     (stroke (width 0) (type default))
   )
-  (wire (pts (xy 74.93 87.63) (xy 78.74 87.63))
+  (wire (pts (xy 74.93 82.55) (xy 78.74 82.55))
     (stroke (width 0) (type default))
   )
@@
     (stroke (width 0) (type default))
   )
-  (wire (pts (xy 78.74 82.55) (xy 78.74 87.63))
+  (wire (pts (xy 78.74 77.47) (xy 78.74 82.55))
     (stroke (width 0) (type default))
   )
@@
       (effects (font (size 1.27 1.27)))
     )
-    (property "Footprint" "Button_Switch_SMD:DEALON_MK-12D04-G2" (at 69.85 85.09 0)
+    (property "Footprint" "easyeda2kicad:SW-TH_MSK12C02" (at 69.85 85.09 0)
       (effects (font (size 1.27 1.27)) hide)
     )
@@
     )
   )
-  (symbol (lib_id "power:GND") (at 83.82 92.71 0) (unit 1)
-    (in_bom yes) (on_board yes) (dnp no) (fields_autoplaced)
-    (property "Reference" "#PWR03" (at 83.82 99.06 0)
-      (effects (font (size 1.27 1.27)) hide)
-    )
-    (property "Value" "GND" (at 83.82 96.8455 0)
-      (effects (font (size 1.27 1.27)))
-    )
-    (property "Footprint" "" (at 83.82 92.71 0)
-      (effects (font (size 1.27 1.27)) hide)
-    )
-    (property "Datasheet" "" (at 83.82 92.71 0)
+  (symbol (lib_id "power:GND") (at 83.82 87.63 0) (unit 1)
+    (in_bom yes) (on_board yes) (dnp no) (fields_autoplaced)
+    (property "Reference" "#PWR03" (at 83.82 93.98 0)
+      (effects (font (size 1.27 1.27)) hide)
+    )
+    (property "Value" "GND" (at 83.82 91.7655 0)
+      (effects (font (size 1.27 1.27)))
+    )
+    (property "Footprint" "" (at 83.82 87.63 0)
+      (effects (font (size 1.27 1.27)) hide)
+    )
+    (property "Datasheet" "" (at 83.82 87.63 0)
       (effects (font (size 1.27 1.27)) hide)
     )
@@
     )
   )
-  (symbol (lib_id "power:VCC") (at 78.74 82.55 0) (unit 1)
-    (in_bom yes) (on_board yes) (dnp no) (fields_autoplaced)
-    (property "Reference" "#PWR02" (at 78.74 86.36 0)
-      (effects (font (size 1.27 1.27)) hide)
-    )
-    (property "Value" "VCC" (at 78.74 79.0481 0)
-      (effects (font (size 1.27 1.27)))
-    )
-    (property "Footprint" "" (at 78.74 82.55 0)
-      (effects (font (size 1.27 1.27)) hide)
-    )
-    (property "Datasheet" "" (at 78.74 82.55 0)
+  (symbol (lib_id "power:VCC") (at 78.74 77.47 0) (unit 1)
+    (in_bom yes) (on_board yes) (dnp no) (fields_autoplaced)
+    (property "Reference" "#PWR02" (at 78.74 81.28 0)
+      (effects (font (size 1.27 1.27)) hide)
+    )
+    (property "Value" "VCC" (at 78.74 73.9681 0)
+      (effects (font (size 1.27 1.27)))
+    )
+    (property "Footprint" "" (at 78.74 77.47 0)
+      (effects (font (size 1.27 1.27)) hide)
+    )
+    (property "Datasheet" "" (at 78.74 77.47 0)
       (effects (font (size 1.27 1.27)) hide)
     )
@@
       (effects (font (size 1.27 1.27)) (justify left))
     )
-    (property "Footprint" "Battery:BatteryHolder_Keystone_3002_1x2032" (at 57.15 88.646 90)
+    (property "Footprint" "easyeda2kicad:BAT-SMD_CR2032-3V" (at 57.15 88.646 90)
       (effects (font (size 1.27 1.27)) hide)
     )
@@
     )
   )
-  (symbol (lib_id "Device:C_Small") (at 83.82 90.17 0) (unit 1)
-    (in_bom yes) (on_board yes) (dnp no) (fields_autoplaced)
-    (property "Reference" "C1" (at 86.1441 89.5326 0)
+  (symbol (lib_id "Device:C_Small") (at 83.82 85.09 0) (unit 1)
+    (in_bom yes) (on_board yes) (dnp no) (fields_autoplaced)
+    (property "Reference" "C1" (at 86.1441 84.4526 0)
       (effects (font (size 1.27 1.27)) (justify left))
     )
-    (property "Value" "100nF" (at 86.1441 91.4536 0)
+    (property "Value" "100nF" (at 86.1441 86.3736 0)
       (effects (font (size 1.27 1.27)) (justify left))
     )
-    (property "Footprint" "Capacitor_SMD:C_0603_1608Metric_Pad1.08x0.95mm_HandSolder" (at 83.82 90.17 0)
-      (effects (font (size 1.27 1.27)) hide)
-    )
-    (property "Datasheet" "~" (at 83.82 90.17 0)
-      (effects (font (size 1.27 1.27)) hide)
-    )
+    (property "Footprint" "Capacitor_SMD:C_0603_1608Metric_Pad1.08x0.95mm_HandSolder" (at 83.82 85.09 0)
+      (effects (font (size 1.27 1.27)) hide)
+    )
+    (property "Datasheet" "~" (at 83.82 85.09 0)
+      (effects (font (size 1.27 1.27)) hide)
+    )

Commit message: Generated Output-Files, Added LCSC-Partnumbers to schematic
Parts:
- BT1: LCSC (none) -> C70373
- C1: LCSC (none) -> C38141
- D1: LCSC (none) -> C396649
- D2, D3, D4, D5, D6: LCSC (none) -> C965799
- R1, R2, R3, R4, R6, R7: LCSC (none) -> C5140946
- R5: LCSC (none) -> C3016757
- SW1: LCSC (none) -> C2681568
- U1: LCSC (none) -> C189365
Changed lines of the file:
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@@
+      (effects (font (size 1.27 1.27)) hide)
+    )
+    (property "LCSC" "C965799" (at 166.37 107.95 90)
       (effects (font (size 1.27 1.27)) hide)
     )
@@
       (effects (font (size 1.27 1.27)) hide)
     )
+    (property "LCSC" "C2681568" (at 69.85 85.09 0)
+      (effects (font (size 1.27 1.27)) hide)
+    )
     (pin "1")
     (pin "2")
@@
       (effects (font (size 1.27 1.27)) hide)
     )
+    (property "LCSC" "C5140946" (at 193.04 102.87 0)
+      (effects (font (size 1.27 1.27)) hide)
+    )
     (pin "1")
     (pin "2")
@@
       (effects (font (size 1.27 1.27)) hide)
     )
+    (property "LCSC" "C3016757" (at 191.77 85.09 90)
+      (effects (font (size 1.27 1.27)) hide)
+    )
     (pin "1")
     (pin "2")
@@
       (effects (font (size 1.27 1.27)) hide)
     )
+    (property "LCSC" "C965799" (at 128.27 107.95 90)
+      (effects (font (size 1.27 1.27)) hide)
+    )
     (pin "1")
     (pin "2")
@@
     )
     (property "Datasheet" "~" (at 205.74 107.95 90)
+      (effects (font (size 1.27 1.27)) hide)
+    )
+    (property "LCSC" "C965799" (at 205.74 107.95 90)
       (effects (font (size 1.27 1.27)) hide)
     )
@@
       (effects (font (size 1.27 1.27)) hide)
     )
+    (property "LCSC" "C70373" (at 57.15 90.17 0)
+      (effects (font (size 1.27 1.27)) hide)
+    )
     (pin "1")
     (pin "2")
@@
     )
     (property "Datasheet" "~" (at 128.27 102.87 0)
+      (effects (font (size 1.27 1.27)) hide)
+    )
+    (property "LCSC" "C5140946" (at 128.27 102.87 0)
       (effects (font (size 1.27 1.27)) hide)
     )
@@
     )
     (property "Datasheet" "http://ww1.microchip.com/downloads/en/DeviceDoc/40001912A.pdf" (at 151.13 92.71 0)
+      (effects (font (size 1.27 1.27)) hide)
+    )
+    (property "LCSC" "C189365" (at 151.13 92.71 0)
       (effects (font (size 1.27 1.27)) hide)
     )
@@
   )
   (symbol (lib_id "Device:C_Small") (at 83.82 85.09 0) (unit 1)
-    (in_bom yes) (on_board yes) (dnp no) (fields_autoplaced)
+    (in_bom yes) (on_board yes) (dnp no)
     (property "Reference" "C1" (at 86.1441 84.4526 0)
       (effects (font (size 1.27 1.27)) (justify left))
@@
       (effects (font (size 1.27 1.27)) hide)
     )
+    (property "LCSC" "C38141" (at 83.82 85.09 0)
+      (effects (font (size 1.27 1.27)) hide)
+    )
     (pin "1")
     (pin "2")
@@
     )
     (property "Datasheet" "~" (at 180.34 107.95 90)
+      (effects (font (size 1.27 1.27)) hide)
+    )
+    (property "LCSC" "C965799" (at 180.34 107.95 90)
       (effects (font (size 1.27 1.27)) hide)
     )
@@
       (effects (font (size 1.27 1.27)) hide)
     )
+    (property "LCSC" "C5140946" (at 180.34 102.87 0)
+      (effects (font (size 1.27 1.27)) hide)
+    )
     (pin "1")
     (pin "2")
@@
       (effects (font (size 1.27 1.27)) hide)
     )
+    (property "LCSC" "C396649" (at 115.57 107.95 90)
+      (effects (font (size 1.27 1.27)) hide)
+    )
     (pin "1")
     (pin "2")
@@
     )
     (property "Datasheet" "~" (at 193.04 107.95 90)
+      (effects (font (size 1.27 1.27)) hide)
+    )
+    (property "LCSC" "C965799" (at 193.04 107.95 90)
       (effects (font (size 1.27 1.27)) hide)
     )
@@
       (effects (font (size 1.27 1.27)) hide)
     )
+    (property "LCSC" "C5140946" (at 205.74 102.87 0)
+      (effects (font (size 1.27 1.27)) hide)
+    )
     (pin "1")
     (pin "2")
@@
       (effects (font (size 1.27 1.27)) hide)
     )
+    (property "LCSC" "C5140946" (at 166.37 102.87 0)
+      (effects (font (size 1.27 1.27)) hide)
+    )
     (pin "1")
     (pin "2")
@@
       (effects (font (size 1.27 1.27)) hide)
     )
+    (property "LCSC" "C5140946" (at 115.57 102.87 0)
+      (effects (font (size 1.27 1.27)) hide)
+    )

Commit message: minor fixes
Parts:
- R5: LCSC C3016757 -> C5140946
Changed lines of the file:
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@@
       (effects (font (size 1.27 1.27)) hide)
     )
-    (property "LCSC" "C3016757" (at 191.77 85.09 90)
+    (property "LCSC" "C5140946" (at 191.77 85.09 90)
       (effects (font (size 1.27 1.27)) hide)
     )

Commit message: Replaced all footprints exept 0603-resistor with LCSC-footprints, generated new production-files, replaced 0805-cap with 0603-cap inside materialliste
Parts:
- C1: footprint Capacitor_SMD:C_0603_1608Metric_Pad1.08x0.95mm_HandSolder -> easyeda2kicad:C0603
- D1: footprint LED_SMD:LED_1206_3216Metric -> easyeda2kicad:LED-SMD_L3.2-W2.1-R-FD
- D2, D3, D4, D5, D6: footprint LED_SMD:LED_0603_1608Metric -> easyeda2kicad:LED0603-RD_RED
- U1: footprint Package_SO:SOIC-14_3.9x8.7mm_P1.27mm -> easyeda2kicad:SOIC-14_L8.7-W3.9-P1.27-LS6.0-BL
Changed lines of the file:
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@@
       (effects (font (size 1.27 1.27)) (justify right))
     )
-    (property "Footprint" "LED_SMD:LED_0603_1608Metric" (at 166.37 107.95 90)
+    (property "Footprint" "easyeda2kicad:LED0603-RD_RED" (at 166.37 107.95 90)
       (effects (font (size 1.27 1.27)) hide)
     )
@@
       (effects (font (size 1.27 1.27)) (justify right))
     )
-    (property "Footprint" "LED_SMD:LED_0603_1608Metric" (at 128.27 107.95 90)
+    (property "Footprint" "easyeda2kicad:LED0603-RD_RED" (at 128.27 107.95 90)
       (effects (font (size 1.27 1.27)) hide)
     )
@@
       (effects (font (size 1.27 1.27)) (justify right))
     )
-    (property "Footprint" "LED_SMD:LED_0603_1608Metric" (at 205.74 107.95 90)
+    (property "Footprint" "easyeda2kicad:LED0603-RD_RED" (at 205.74 107.95 90)
       (effects (font (size 1.27 1.27)) hide)
     )
@@
       (effects (font (size 1.27 1.27)) (justify left))
     )
-    (property "Footprint" "Package_SO:SOIC-14_3.9x8.7mm_P1.27mm" (at 151.13 92.71 0)
+    (property "Footprint" "easyeda2kicad:SOIC-14_L8.7-W3.9-P1.27-LS6.0-BL" (at 151.13 92.71 0)
       (effects (font (size 1.27 1.27) italic) hide)
     )
@@
       (effects (font (size 1.27 1.27)) (justify left))
     )
-    (property "Footprint" "Capacitor_SMD:C_0603_1608Metric_Pad1.08x0.95mm_HandSolder" (at 83.82 85.09 0)
+    (property "Footprint" "easyeda2kicad:C0603" (at 83.82 85.09 0)
       (effects (font (size 1.27 1.27)) hide)
     )
@@
       (effects (font (size 1.27 1.27)) (justify right))
     )
-    (property "Footprint" "LED_SMD:LED_0603_1608Metric" (at 180.34 107.95 90)
+    (property "Footprint" "easyeda2kicad:LED0603-RD_RED" (at 180.34 107.95 90)
       (effects (font (size 1.27 1.27)) hide)
     )
@@
       (effects (font (size 1.27 1.27)) (justify right))
     )
-    (property "Footprint" "LED_SMD:LED_1206_3216Metric" (at 115.57 107.95 90)
+    (property "Footprint" "easyeda2kicad:LED-SMD_L3.2-W2.1-R-FD" (at 115.57 107.95 90)
       (effects (font (size 1.27 1.27)) hide)
     )
@@
       (effects (font (size 1.27 1.27)) (justify right))
     )
-    (property "Footprint" "LED_SMD:LED_0603_1608Metric" (at 193.04 107.95 90)
-      (effects (font (size 1.27 1.27)) hide)
-    )
+    (property "Footprint" "easyeda2kicad:LED0603-RD_RED" (at 193.04 107.95 90)
+      (effects (font (size 1.27 1.27)) hide)
+    )

Commit message: removed clk-pad from pcb, increased size of rothli-sticker, change IR-diode resistor from 590 to 220
Parts:
- removed J4: EXTCLK, TestPoint:TestPoint_Pad_D2.0mm, symbol Connector:Conn_01x01_Pin
- R5: value 590 -> 220
Connections:
- net EXTCLK: no longer names the net of U1.13 (PA3)
- no-connect marks 1 -> 2
Changed lines of the file:
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@@
   )
   (no_connect (at 74.93 87.63))
+  (no_connect (at 166.37 90.17))
   (wire (pts (xy 181.61 82.55) (xy 166.37 82.55))
     (stroke (width 0) (type default))
@@
     (stroke (width 0) (type default))
   )
-  (wire (pts (xy 166.37 90.17) (xy 181.61 90.17))
-    (stroke (width 0) (type default))
-  )
   (wire (pts (xy 57.15 85.09) (xy 64.77 85.09))
     (stroke (width 0) (type default))
@@
   )
   (label "LED 3" (at 167.64 97.79 0) (fields_autoplaced)
-    (effects (font (size 1.27 1.27)) (justify left bottom))
-  )
-  (label "EXTCLK" (at 167.64 90.17 0) (fields_autoplaced)
     (effects (font (size 1.27 1.27)) (justify left bottom))
   )
@@
       (effects (font (size 1.27 1.27)))
     )
-    (property "Value" "590" (at 191.77 82.55 90)
+    (property "Value" "220" (at 191.77 82.55 90)
       (effects (font (size 1.27 1.27)))
     )
@@
         )
       )
-    )
-  )
-  (symbol (lib_id "Connector:Conn_01x01_Pin") (at 186.69 90.17 180) (unit 1)
-    (in_bom yes) (on_board yes) (dnp no)
-    (property "Reference" "J4" (at 186.69 88.9 0)
-      (effects (font (size 1.27 1.27)))
-    )
-    (property "Value" "EXTCLK" (at 173.99 88.9 0)
-      (effects (font (size 1.27 1.27)) (justify left) hide)
-    )
-    (property "Footprint" "TestPoint:TestPoint_Pad_D2.0mm" (at 186.69 90.17 0)
-      (effects (font (size 1.27 1.27)) hide)
-    )
-    (property "Datasheet" "~" (at 186.69 90.17 0)
-      (effects (font (size 1.27 1.27)) hide)
-    )
-    (pin "1")
-    (instances
-      (project "ET-Abschlussgadget_2023"
-        (path "/175a65ba-6b59-4269-bd86-2662d331b61e"
-          (reference "J4") (unit 1)
-        )
-      )

Commit message: Add ground plane pattern to entire back side
Connections:
- net Cap_Pad / ADC1: no longer U1.12 (PA2)
- no-connect marks 2 -> 3
Changed lines of the file:
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@@
   (junction (at 195.58 85.09) (diameter 0) (color 0 0 0 0)
   )
-  (junction (at 187.96 85.09) (diameter 0) (color 0 0 0 0)
-  )
+  (no_connect (at 166.37 87.63))
   (no_connect (at 74.93 87.63))
   (no_connect (at 166.37 90.17))
@@
     (stroke (width 0) (type default))
   )
-  (wire (pts (xy 166.37 87.63) (xy 187.96 87.63))
-    (stroke (width 0) (type default))
-  )
   (wire (pts (xy 193.04 95.25) (xy 193.04 100.33))
     (stroke (width 0) (type default))
@@
     (stroke (width 0) (type default))
   )
-  (wire (pts (xy 189.23 85.09) (xy 187.96 85.09))
+  (wire (pts (xy 166.37 85.09) (xy 189.23 85.09))
     (stroke (width 0) (type default))
   )
@@
   )
   (wire (pts (xy 78.74 82.55) (xy 83.82 82.55))
-    (stroke (width 0) (type default))
-  )
-  (wire (pts (xy 187.96 85.09) (xy 166.37 85.09))
-    (stroke (width 0) (type default))
-  )
-  (wire (pts (xy 187.96 85.09) (xy 187.96 87.63))
     (stroke (width 0) (type default))
   )
@@
     (effects (font (size 1.27 1.27)) (justify left bottom))
   )
-  (label "Cap_Pad {slash} ADC2" (at 167.64 87.63 0) (fields_autoplaced)
-    (effects (font (size 1.27 1.27)) (justify left bottom))
-  )

Commit message: Updated schematic with MOSFET and pulldown resistors, changed footprint for IR-diode
Parts:
- added Q1: NMOS, easyeda2kicad:SOT-23-3_L2.9-W1.3-P1.90-LS2.4-BR, symbol Simulation_SPICE:NMOS
- added R8: 1M, Resistor_SMD:R_0603_1608Metric_Pad0.98x0.95mm_HandSolder, symbol Device:R_Small
- D1: footprint easyeda2kicad:LED-SMD_L3.2-W2.1-R-FD -> Diode_SMD:XS-IR04A05-802
- R1: value 590 -> 100k
- renumbered J5 to J1, J6 to J2, J1 to J3, J2 to J4, J3 to J5
Connections:
- net Cap_Pad: now also R8.2
- net GND: now also R1.1, Q1.3 (S), R8.1; no longer D1.1 (K)
- net LED IR: now also Q1.2 (G)
- net VCC: now also D1.2 (A)
- new net: D1.1 (K), Q1.1 (D)
Other:
- moved on the sheet: D1
