File: ET-Abschlussgadget_2023/ET-Abschlussgadget_2023.kicad_sch (KiCad schematic)
At the start: 25 parts, among them J1 EXTCLK, J2 EXTCLK, J3 PB0, J4 PB1, J5 UPDI / RESET, Q1 NMOS, SW1 ON/OFF, U1 ATtiny414-SS

Commit message: Remove pulldown, Update resistors, Update routing
Parts:
- removed R1: 100k, Resistor_SMD:R_0603_1608Metric_Pad0.98x0.95mm_HandSolder, symbol Device:R_Small
- R2, R3, R4, R6, R7: value 590 -> 560
- R5: value 220 -> 560
Connections:
- net Cap_Pad: no longer R8.2
- net Cap_Pad / ADC1: now also R8.2, U1.13 (PA3); no longer U1.11 (PA1)
Other:
- moved on the sheet: R5, R8, TP1

Commit message: Replaced parts in materialliste, replaced some footprints, generade production-files with JLC-plugin
Parts:
- removed Q1: NMOS, easyeda2kicad:SOT-23-3_L2.9-W1.3-P1.90-LS2.4-BR, symbol Simulation_SPICE:NMOS
- added Q1: SI2302_C2891732, easyeda2kicad:SOT-23-3_L2.9-W1.3-P1.90-LS2.4-BR, symbol easyeda2kicad:SI2302_C2891732
- D1: LCSC C396649 -> C5205266
- R1: renamed from R2; LCSC C5140946 -> C25247
- R2: renamed from R3; LCSC C5140946 -> C25247
- R3: renamed from R4; LCSC C5140946 -> C25247
- R4: renamed from R6; LCSC C5140946 -> C25247
- R5: renamed from R7; LCSC C5140946 -> C25247
- R6: renamed from R8; LCSC C5140946 -> C3152128
- R7: renamed from R5; LCSC C5140946 -> C25247
Connections:
- net GND: now also Q1.2 (S)
- net LED IR: now also Q1.1 (G)
- net at D1.1 (K): now also Q1.3 (D)
