File: ET-Abschlussgadget_2023/ET-Abschlussgadget_2023-rounded.kicad_pcb (KiCad board)
At the start: 2 copper layers, 85 x 54 mm, 37 parts, among them J1 EXTCLK, J2 EXTCLK, J3 PB0, J4 PB1, J5 UPDI / RESET, Q2 SI2302_C2891732, SW1 ON/OFF, U1 ATtiny414-SS

Commit message: Final export
Parts:
- moved R8 0.92 mm to (137.6, 102.0), turned to 0 degrees
- moved R5 0.70 mm to (137.6, 100.0)
Routing:
- net /Cap_Pad / ADC1: track 9.74 -> 7.18 mm
- net /Cap_Pad: track 11.1 -> 11.8 mm
Other:
- board text added: "uint8_t avgAge = 25;"
- board text removed: "uint16_t avgAge = 25;"
